Commit message: colour,worlds,teleop

File: src/heyrobo_description/urdf/heyrobo.xacro (robot description, xacro)
@@ -3,5 +3,7 @@
 <xacro:include filename="$(find heyrobo_description)/urdf/materials.xacro" />
 <xacro:include filename="$(find heyrobo_description)/urdf/heyrobo.trans" />
-<xacro:include filename="$(find heyrobo_description)/urdf/heyrobo.gazebo" />
+<xacro:include filename="$(find heyrobo_description)/gazebo/heyrobo_material.gazebo" />
+<xacro:include filename="$(find heyrobo_description)/gazebo/heyrobo_physics.gazebo" />
+<xacro:include filename="$(find heyrobo_description)/gazebo/heyrobo_plugins.gazebo" />
 <link name="base_link">
   <inertial>
@@ -15,5 +17,5 @@
       <mesh filename="package://heyrobo_description/meshes/base_link.stl" scale="0.001 0.001 0.001"/>
     </geometry>
-    <material name="silver"/>
+    <material name="FlatBlack"/>
   </visual>
   <collision>
@@ -35,5 +37,5 @@
       <mesh filename="package://heyrobo_description/meshes/wheel_left_1.stl" scale="0.001 0.001 0.001"/>
     </geometry>
-    <material name="silver"/>
+    <material name="Black"/>
   </visual>
   <collision>
@@ -55,5 +57,5 @@
       <mesh filename="package://heyrobo_description/meshes/wheel_right_1.stl" scale="0.001 0.001 0.001"/>
     </geometry>
-    <material name="silver"/>
+    <material name="Black"/>
   </visual>
   <collision>
@@ -75,5 +77,5 @@
       <mesh filename="package://heyrobo_description/meshes/buck_converter_1.stl" scale="0.001 0.001 0.001"/>
     </geometry>
-    <material name="silver"/>
+    <material name="Orange"/>
   </visual>
   <collision>
@@ -95,5 +97,5 @@
       <mesh filename="package://heyrobo_description/meshes/caster_forward_1.stl" scale="0.001 0.001 0.001"/>
     </geometry>
-    <material name="silver"/>
+    <material name="White"/>
   </visual>
   <collision>
@@ -115,5 +117,5 @@
       <mesh filename="package://heyrobo_description/meshes/motor_left_1.stl" scale="0.001 0.001 0.001"/>
     </geometry>
-    <material name="silver"/>
+    <material name="Yellow"/>
   </visual>
   <collision>
@@ -135,5 +137,5 @@
       <mesh filename="package://heyrobo_description/meshes/motor_right_1.stl" scale="0.001 0.001 0.001"/>
     </geometry>
-    <material name="silver"/>
+    <material name="Yellow"/>
   </visual>
   <collision>
@@ -155,5 +157,5 @@
       <mesh filename="package://heyrobo_description/meshes/motordriver_1.stl" scale="0.001 0.001 0.001"/>
     </geometry>
-    <material name="silver"/>
+    <material name="Orange"/>
   </visual>
   <collision>
@@ -175,5 +177,5 @@
       <mesh filename="package://heyrobo_description/meshes/caster_backward_1.stl" scale="0.001 0.001 0.001"/>
     </geometry>
-    <material name="silver"/>
+    <material name="White"/>
   </visual>
   <collision>
@@ -195,5 +197,5 @@
       <mesh filename="package://heyrobo_description/meshes/jetson_nano_1.stl" scale="0.001 0.001 0.001"/>
     </geometry>
-    <material name="silver"/>
+    <material name="Green"/>
   </visual>
   <collision>
@@ -215,5 +217,5 @@
       <mesh filename="package://heyrobo_description/meshes/charger_module_1.stl" scale="0.001 0.001 0.001"/>
     </geometry>
-    <material name="silver"/>
+    <material name="Red"/>
   </visual>
   <collision>
@@ -235,5 +237,5 @@
       <mesh filename="package://heyrobo_description/meshes/mpu_1.stl" scale="0.001 0.001 0.001"/>
     </geometry>
-    <material name="silver"/>
+    <material name="Red"/>
   </visual>
   <collision>
@@ -255,5 +257,5 @@
       <mesh filename="package://heyrobo_description/meshes/depth_camera_1.stl" scale="0.001 0.001 0.001"/>
     </geometry>
-    <material name="silver"/>
+    <material name="Blue"/>
   </visual>
   <collision>
@@ -275,5 +277,5 @@
       <mesh filename="package://heyrobo_description/meshes/lidar_1.stl" scale="0.001 0.001 0.001"/>
     </geometry>
-    <material name="silver"/>
+    <material name="Black"/>
   </visual>
   <collision>

File: src/heyrobo_description/urdf/materials.xacro (robot description, xacro)
@@ -1,6 +1,27 @@
 <?xml version="1.0" ?>
 <robot name="heyrobo" xmlns:xacro="http://www.ros.org/wiki/xacro" >
-<material name="silver">
-  <color rgba="0.700 0.700 0.700 1.000"/>
+<material name="FlatBlack">
+  <color rgba="0.184 0.184 0.184 1.000"/>
+</material>
+<material name="Black">
+  <color rgba="0 0 0 1.000"/>
+</material>
+<material name="Orange">
+  <color rgba="0.8 0.4 0.0 1.000"/>
+</material>
+<material name="White">
+  <color rgba="1 1 1 1.000"/>
+</material>
+<material name="Yellow">
+  <color rgba="1 1 0 1.000"/>
+</material>
+<material name="Green">
+  <color rgba="0 0.5 0 1.000"/>
+</material>
+<material name="Red">
+  <color rgba="1 0 0 1.000"/>
+</material>
+<material name="Blue">
+  <color rgba="0 0 1 1.000"/>
 </material>
 </robot>
